File: MYNDberry/MYNDberry.kicad_sch (KiCad schematic)
At the start: 31 parts, among them CN1 1.0-4P WT, J1 Power Header, J2 Audio Header, J3 MCU/Debug Header, J4 RPi Peripheral Header, J5 Conn_01x09, J6 Conn_01x09, J7 I2S Header, J8 Conn_01x03, Q1 AO3400A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

Commit message: Created new version using through hole headers for RasPi
Parts:
- removed H2: RPi, Library:2x40_2.54mm_Female_SMT_Vertical, symbol Library:PM254-2-20-WS-8.5
- added U3: HC-PM254-8.5H-2X20PW, Library:HDR-TH_40P-P2.54-H-F-R2-C20-S2.54-N, symbol MYNDberry:HC-PM254-8.5H-2X20PW
- C1, C2, C3: symbol Library:C -> MYNDberry:C
- CN1: symbol Library:1.0-4PWT -> MYNDberry:1.0-4PWT
- H1: symbol Library:XDZ254-2-12-S-2.5-G1 -> MYNDberry:XDZ254-2-12-S-2.5-G1
- H3: symbol Library:HXPZ2.54-1X3PWT -> MYNDberry:HXPZ2.54-1X3PWT
- J1, J2, J3, J4, J7: symbol Library:Conn_02x04_Odd_Even -> MYNDberry:Conn_02x04_Odd_Even
- J5, J6: symbol Library:Conn_01x09 -> MYNDberry:Conn_01x09
- J8: symbol Library:Conn_01x03 -> MYNDberry:Conn_01x03
- Q1: symbol Library:AO3400A -> MYNDberry:AO3400A
- Q2: symbol Library:AO3401A -> MYNDberry:AO3401A
- R1, R10, R11, R12, R2, R3, R4, R5, R6, R7, R8, R9: symbol Library:R_US -> MYNDberry:R_US
- U1: symbol Library:TPS70933DBVR -> MYNDberry:TPS70933DBVR
- U2: symbol Library:CH340N_C2977777 -> MYNDberry:CH340N_C2977777
Connections:
- net 5V_RPi: now also U3.2, U3.4
- net CE0: now also U3.24
- net CE1: now also U3.26
- net GND: now also U3.14, U3.20, U3.25, U3.30, U3.34, U3.39, U3.6, U3.9
- net GPIO_0: now also U3.27
- net GPIO_1: now also U3.28
- net GPIO_12: now also U3.32
- net GPIO_13: now also U3.33
- net GPIO_16: now also U3.36
- net GPIO_17: now also U3.11
- net GPIO_22: now also U3.15
- net GPIO_23: now also U3.16
- net GPIO_24: now also U3.18
- net GPIO_25: now also U3.22
- net GPIO_26: now also U3.37
- net GPIO_27: now also U3.13
- net GPIO_4: now also U3.7
- net GPIO_5: now also U3.29
- net GPIO_6: now also U3.31
- net I2C1_SCL: now also U3.5
- net I2C1_SDA: now also U3.3
- net I2S_BCLK: now also U3.12
- net I2S_DIN: now also U3.38
- net I2S_DOUT: now also U3.40
- net I2S_WCLK: now also U3.35
- net MISO: now also U3.21
- net MOSI: now also U3.19
- net SCLK: now also U3.23
- net UART0_RX: now also U3.10
- net UART0_TX: now also U3.8
- new net 3.3V_RPi_1: U3.1
- new net 3.3V_RPi_2: U3.17
